File: KiCad_Lawn_Mower/KiCad_Lawn_Mower.kicad_sch (KiCad schematic)
At the start: 0 parts

Commit message: Kicad updates
Other:
- added sheet ESP32 Pinout (esp32.kicad_sch)
- added sheet IR Sensor Schematic (ir_sensor_schematic.kicad_sch)
- note added: "ESP32-S3"
- note added: "IR Sensor"
Changed lines of the file:
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@@
 	(generator_version "10.0")
 	(paper "A4")
+	(rectangle
+		(start 31.75 29.21)
+		(end 71.12 48.26)
+		(stroke
+			(width 0)
+			(type default)
+		)
+		(fill
+			(type none)
+		)
+	)
+	(rectangle
+		(start 124.46 81.28)
+		(end 182.88 118.11)
+		(stroke
+			(width 0)
+			(type default)
+		)
+		(fill
+			(type none)
+		)
+	)
+	(text "IR Sensor\n"
+		(exclude_from_sim no)
+		(at 51.816 39.116 0)
+		(effects
+			(font
+				(size 5.08 5.08)
+			)
+		)
+	)
+	(text "ESP32-S3"
+		(exclude_from_sim no)
+		(at 153.67 98.806 0)
+		(effects
+			(font
+				(size 6.985 6.985)
+			)
+		)
+	)
+	(sheet
+		(at 31.75 29.21)
+		(size 39.37 19.05)
+		(exclude_from_sim no)
+		(in_bom yes)
+		(on_board yes)
+		(dnp no)
+		(fields_autoplaced yes)
+		(stroke
+			(width 0.1524)
+			(type solid)
+		)
+		(fill
+			(color 0 0 0 0)
+		)
+		(property "Sheetname" "IR Sensor Schematic"
+			(at 31.75 28.4984 0)
+			(show_name no)
+			(do_not_autoplace no)
+			(effects
+				(font
+					(size 1.27 1.27)
+				)
+				(justify left bottom)
+			)
+		)
+		(property "Sheetfile" "ir_sensor_schematic.kicad_sch"
+			(at 31.75 48.8446 0)
+			(show_name no)
+			(do_not_autoplace no)
+			(effects
+				(font
+					(size 1.27 1.27)
+				)
+				(justify left top)
+			)
+		)
+		(instances
+			(project "KiCad_Lawn_Mower"
+				(path "/0806a8c0-bc45-48da-a5f3-b40d8c386964"
+					(page "2")
+				)
+			)
+		)
+	)
+	(sheet
+		(at 124.46 81.28)
+		(size 58.42 36.83)
+		(exclude_from_sim no)
+		(in_bom yes)
+		(on_board yes)
+		(dnp no)
+		(fields_autoplaced yes)
+		(stroke
+			(width 0.1524)
+			(type solid)
+		)
+		(fill
+			(color 0 0 0 0)
+		)
+		(property "Sheetname" "ESP32 Pinout"
+			(at 124.46 80.5684 0)
+			(show_name no)
+			(do_not_autoplace no)
+			(effects
+				(font
+					(size 1.27 1.27)
+				)
+				(justify left bottom)
+			)
+		)
+		(property "Sheetfile" "esp32.kicad_sch"
+			(at 124.46 118.6946 0)
+			(show_name no)
+			(do_not_autoplace no)
+			(effects
+				(font
+					(size 1.27 1.27)
+				)
+				(justify left top)
+			)
+		)
+		(instances
+			(project "KiCad_Lawn_Mower"
+				(path "/0806a8c0-bc45-48da-a5f3-b40d8c386964"
+					(page "3")
+				)
+			)
+		)
+	)
 	(sheet_instances
 		(path "/"

Commit message: Uart init
Other:
- added sheet RPi4 (RPi4.kicad_sch)
- note added: "RPi4"
Changed lines of the file:
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@@
+		)
+	)
+	(text "RPi4"
+		(exclude_from_sim no)
+		(at 74.168 153.67 0)
+		(effects
+			(font
+				(size 6.985 6.985)
+			)
 		)
 	)
@@
 				)
 			)
+		)
+	)
+	(sheet
+		(at 44.45 137.16)
+		(size 57.15 33.02)
+		(exclude_from_sim no)
+		(in_bom yes)
+		(on_board yes)
+		(dnp no)
+		(fields_autoplaced yes)
+		(stroke
+			(width 0.1524)
+			(type solid)
+		)
+		(fill
+			(color 0 0 0 0)
+		)
+		(property "Sheetname" "RPi4"
+			(at 44.45 136.4484 0)
+			(show_name no)
+			(do_not_autoplace no)
+			(effects
+				(font
+					(size 1.27 1.27)
+				)
+				(justify left bottom)
+			)
+		)
+		(property "Sheetfile" "RPi4.kicad_sch"
+			(at 44.45 170.7646 0)
+			(show_name no)
+			(do_not_autoplace no)
+			(effects
+				(font
+					(size 1.27 1.27)
+				)
+				(justify left top)
+			)
+		)
+		(instances
+			(project "KiCad_Lawn_Mower"
+				(path "/0806a8c0-bc45-48da-a5f3-b40d8c386964"
+					(page "4")
+				)
+			)
